File: BF-AVR/BF-AVR.kicad_sch (KiCad schematic)
At the start: 7 parts, among them J1 USB_B, U2 ATmega1284P PPU, Y2 16MHz

Commit message: a
Parts:
- removed C6, C7: 22pF, symbol Device:C
- removed U2: ATmega1284P PPU, Package_DIP:DIP-40_W15.24mm, symbol MCU_Microchip_ATmega:ATmega1284P-P
- removed Y2: 16MHz, symbol Device:Crystal
- added C2: 0.1μF, Capacitor_THT:C_Disc_D3.0mm_W2.0mm_P2.50mm, symbol Device:C
- added C4, C5: 22pF, Capacitor_THT:C_Disc_D3.0mm_W2.0mm_P2.50mm, symbol Device:C
- added J10, J11, J13, J14, J2, J3: Conn_01x01_Socket, Connector_PinHeader_1.00mm:PinHeader_1x01_P1.00mm_Vertical, symbol Connector:Conn_01x01_Socket
- added J12: DE15_Socket_HighDensity_MountingHoles, Connector_Dsub:DSUB-15-HD_Socket_Horizontal_P2.29x2.54mm_EdgePinOffset8.35mm_Housed_MountingHolesOffset10.89mm, symbol Connector:DE15_Socket_HighDensity_MountingHoles
- added J15: Mini-DIN-6, symbol Connector:Mini-DIN-6
- added J16: Conn_01x15_Socket, symbol Connector:Conn_01x15_Socket
- added J17: Conn_01x06_Socket, symbol Connector:Conn_01x06_Socket
- added J4, J6, J7: Conn_01x03_Pin, symbol Connector:Conn_01x03_Pin
- added J5: Conn_02x14_Counter_Clockwise, symbol Connector_Generic:Conn_02x14_Counter_Clockwise
- added J8, J9: Conn_01x14_Socket, symbol Connector:Conn_01x14_Socket
- added R1: 10kΩ, Resistor_THT:R_Axial_DIN0207_L6.3mm_D2.5mm_P7.62mm_Horizontal, symbol Device:R
- added SW1: SW_RESET, Button_Switch_THT:SW_PUSH_6mm_H4.3mm, symbol Switch:SW_Push
- C1: renamed from C2; footprint (none) -> Capacitor_THT:C_Disc_D3.0mm_W2.0mm_P2.50mm
- C3: footprint (none) -> Capacitor_THT:C_Disc_D3.0mm_W2.0mm_P2.50mm
Connections:
- net GND: now also C2.1, C4.2, C5.2, J12.0, J14.1 (Pin_1), J5.15 (Pin_15), J5.21 (Pin_21), J9.14 (Pin_14), J9.8 (Pin_8), SW1.2
- net VCC: now also C2.2, J13.1 (Pin_1), J5.14 (Pin_14), J5.20 (Pin_20), J5.6 (Pin_6), J8.14 (Pin_14), J8.6 (Pin_6), J9.9 (Pin_9), R1.1
- net D-: now reaches J1.2 (D-)
- net D-: now also J11.1 (Pin_1)
- net D+: now reaches J1.3 (D+)
- net D+: now also J10.1 (Pin_1)
- new net: C4.1, J2.1 (Pin_1), J6.1 (Pin_1)
- new net: J5.23 (Pin_23), J6.2 (Pin_2)
- new net: J7.3 (Pin_3), R1.2, SW1.1
- new net: J4.2 (Pin_2), J5.22 (Pin_22)
- new net: C5.1, J3.1 (Pin_1), J4.3 (Pin_3)
- new net DIN_1: J15.1, J17.1 (Pin_1)
- new net DIN_2: J15.2, J17.2 (Pin_2)
- new net DIN_3: J15.3, J17.3 (Pin_3)
- new net DIN_4: J15.4, J17.4 (Pin_4)
- new net DIN_5: J15.5, J17.5 (Pin_5)
- new net DIN_6: J15.6, J17.6 (Pin_6)
- new net DSub_1: J12.1, J16.1 (Pin_1)
- new net DSub_10: J12.10, J16.10 (Pin_10)
- new net DSub_11: J12.11, J16.11 (Pin_11)
- new net DSub_12: J12.12, J16.12 (Pin_12)
- new net DSub_13: J12.13, J16.13 (Pin_13)
- new net DSub_14: J12.14, J16.14 (Pin_14)
- new net DSub_15: J12.15, J16.15 (Pin_15)
- new net DSub_2: J12.2, J16.2 (Pin_2)
- new net DSub_3: J12.3, J16.3 (Pin_3)
- new net DSub_4: J12.4, J16.4 (Pin_4)
- new net DSub_5: J12.5, J16.5 (Pin_5)
- new net DSub_6: J12.6, J16.6 (Pin_6)
- new net DSub_7: J12.7, J16.7 (Pin_7)
- new net DSub_8: J12.8, J16.8 (Pin_8)
- new net DSub_9: J12.9, J16.9 (Pin_9)
- new net PA0: J4.1 (Pin_1), J9.7 (Pin_7)
- new net PA1: J6.3 (Pin_3), J9.6 (Pin_6)
- new net PA2: J5.24 (Pin_24), J9.5 (Pin_5)
- new net PA3: J5.25 (Pin_25), J9.4 (Pin_4)
- new net PA4: J5.26 (Pin_26), J9.3 (Pin_3)
- new net PA5: J5.27 (Pin_27), J9.2 (Pin_2)
- new net PA6: J5.28 (Pin_28), J9.1 (Pin_1)
- new net PA7: J5.1 (Pin_1), J8.1 (Pin_1)
- new net PC0: J5.2 (Pin_2), J8.2 (Pin_2)
- new net PC1: J5.3 (Pin_3), J8.3 (Pin_3)
- new net PC2: J5.4 (Pin_4), J8.4 (Pin_4)
- new net PC3: J5.5 (Pin_5), J8.5 (Pin_5)
- new net PD1: J5.7 (Pin_7), J8.7 (Pin_7)
- new net PD2: J5.8 (Pin_8), J8.8 (Pin_8)
- new net PD3: J5.9 (Pin_9), J8.9 (Pin_9)
- new net PD4: J5.10 (Pin_10), J8.10 (Pin_10)
- new net PD5: J5.11 (Pin_11), J8.11 (Pin_11)
- new net PD6: J5.12 (Pin_12), J8.12 (Pin_12)
- new net PD7: J5.13 (Pin_13), J8.13 (Pin_13)
- new net PF0: J5.16 (Pin_16), J9.13 (Pin_13)
- new net PF1: J5.17 (Pin_17), J9.12 (Pin_12)
- new net PF6: J7.1 (Pin_1)
- new net RESET: J5.18 (Pin_18), J7.2 (Pin_2), J9.11 (Pin_11)
- new net UPDI: J5.19 (Pin_19), J9.10 (Pin_10)
- no-connect marks 2 -> 0
Other:
- moved on the sheet: C1, J1
